File: Hardware/IoT_Irrigation_System_PCA/IoT_Irrigation_System_PCA.kicad_pcb (KiCad board)
At the start: 2 copper layers, 73 x 88.1 mm, 19 parts, among them J1 Conn_01x19_Socket, J2 Conn_01x19_Socket, J3 HW-519R4, J4 691137710002, J5 691137710002, J6 691137710002, J7 Jack-DC, Q1 IRLZ34N, U1 LM2575-5.0BT

Commit message: V1.3.18
Parts:
- moved J4 1.00 mm to (130.8, 61.5)
- moved J5 1.00 mm to (120.0, 61.5)
- renumbered J7 to J3, J3 to J7
Connections:
- J7 pad 6: unconnected-(J3-Pin_6-Pad6) -> GND
Routing:
- net GND: track 2.67 -> 6.61 mm, vias 1 -> 2
- net /RS485_B: track 23.9 -> 22.3 mm
- net /PWR_IN: track 139.5 -> 138.5 mm
Other:
- board text added: "+5V"
- board text added: "NEG"
- board text added: "POS"
- board text added: "PWR"
- board text added: "SOLENOID"
