File: Hardware/IoT_Irrigation_System_PCA/IoT_Irrigation_System_PCA.kicad_sch (KiCad schematic)
At the start: 19 parts, among them J1 Conn_01x19_Socket, J2 Conn_01x19_Socket, J3 HW-519R4, J4 691137710002, J5 691137710002, J6 691137710002, J7 Jack-DC, Q1 IRLZ34N, U1 LM2575-5.0BT

Commit message: V1.3.18
Parts:
- renumbered J7 to J3, J3 to J7
Changed lines of the file:
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@@
 		(on_board yes)
 		(dnp no)
-		(property "Reference" "J3"
+		(property "Reference" "J7"
 			(at 200.406 42.672 0)
 			(effects
@@
 			(project ""
 				(path "/e3c74a8b-a9dc-42be-8052-597c494f9481"
-					(reference "J3")
+					(reference "J7")
 					(unit 1)
 				)
@@
 		(dnp no)
 		(fields_autoplaced yes)
-		(property "Reference" "J7"
+		(property "Reference" "J3"
 			(at 39.37 160.02 0)
 			(effects
@@
 			(project ""
 				(path "/e3c74a8b-a9dc-42be-8052-597c494f9481"
-					(reference "J7")
-					(unit 1)
-				)
+					(reference "J3")
+					(unit 1)
+				)
